Commit message: Major update: depth controller works.

File: src/imm/urdf/remus.urdf (robot description, URDF)
Before this commit: robot remus100, 4 links, 3 joints
Links:
- added link lower_wing; visual box size=0.1 .01 .3
- added link upper_wing; visual box size=0.1 .01 .3
- link left_wing: geometry visual box size=0.1 .3 .01
- link right_wing: geometry visual box size=0.1 .3 .01
Joints:
- added joint base_to_lower_wing: type fixed, parent REMUS, child lower_wing, origin xyz=0 0 0
- added joint base_to_upper_wing: type fixed, parent REMUS, child upper_wing, origin xyz=0 0 0
